Commit message: change package mame to custom_locobot_description

File: urdf/arm_cradle.urdf.xacro (robot description, xacro)
@@ -18,5 +18,5 @@
          <geometry>
            <mesh
-            filename="package://interbotix_xslocobot_descriptions/meshes/locobot_meshes/locobot_arm_cradle.stl"
+            filename="package://custom_locobot_description/meshes/locobot_meshes/locobot_arm_cradle.stl"
             scale="0.001 0.001 0.001"/>
          </geometry>
@@ -27,5 +27,5 @@
          <geometry>
            <mesh
-            filename="package://interbotix_xslocobot_descriptions/meshes/locobot_meshes/locobot_arm_cradle.stl"
+            filename="package://custom_locobot_description/meshes/locobot_meshes/locobot_arm_cradle.stl"
             scale="0.001 0.001 0.001"/>
          </geometry>

File: urdf/battery.urdf.xacro (robot description, xacro)
@@ -16,5 +16,5 @@
         <geometry>
           <mesh
-            filename="package://interbotix_xslocobot_descriptions/meshes/locobot_meshes/locobot_battery.stl"
+            filename="package://custom_locobot_description/meshes/locobot_meshes/locobot_battery.stl"
             scale="0.001 0.001 0.001"/>
         </geometry>
@@ -30,5 +30,5 @@
         <geometry>
           <mesh
-            filename="package://interbotix_xslocobot_descriptions/meshes/locobot_meshes/locobot_battery.stl"
+            filename="package://custom_locobot_description/meshes/locobot_meshes/locobot_battery.stl"
             scale="0.001 0.001 0.001"/>
         </geometry>

File: urdf/camera_tower.urdf.xacro (robot description, xacro)
@@ -16,5 +16,5 @@
         <geometry>
           <mesh
-            filename="package://interbotix_xslocobot_descriptions/meshes/locobot_meshes/${base_type}_version/locobot_camera_tower_${camera_tower_size}.stl"
+            filename="package://custom_locobot_description/meshes/locobot_meshes/${base_type}_version/locobot_camera_tower_${camera_tower_size}.stl"
             scale="${mesh_scale}"/>
         </geometry>
@@ -27,5 +27,5 @@
         <geometry>
           <mesh
-            filename="package://interbotix_xslocobot_descriptions/meshes/locobot_meshes/${base_type}_version/locobot_camera_tower_${camera_tower_size}_simple.stl"
+            filename="package://custom_locobot_description/meshes/locobot_meshes/${base_type}_version/locobot_camera_tower_${camera_tower_size}_simple.stl"
             scale="${mesh_scale}"/>
         </geometry>

File: urdf/custom_pan_and_tilt.urdf.xacro (robot description, xacro)
@@ -1,5 +1,5 @@
 <?xml version="1.0" ?>
 <robot xmlns:xacro="http://ros.org/wiki/xacro">
-  <xacro:include filename="$(find interbotix_xslocobot_descriptions)/urdf/zed2.xacro"/>
+  <xacro:include filename="$(find custom_locobot_description)/urdf/zed2.xacro"/>
   <xacro:macro name="custom_pan_and_tilt" params="*origin">
     <joint name="pan" type="revolute">
@@ -26,5 +26,5 @@
         <geometry>
           <mesh
-            filename="package://interbotix_xslocobot_descriptions/meshes/locobot_meshes/locobot_pan.stl"
+            filename="package://custom_locobot_description/meshes/locobot_meshes/locobot_pan.stl"
             scale="0.001 0.001 0.001"/>
         </geometry>
@@ -37,5 +37,5 @@
         <geometry>
           <mesh
-            filename="package://interbotix_xslocobot_descriptions/meshes/locobot_meshes/locobot_pan.stl"
+            filename="package://custom_locobot_description/meshes/locobot_meshes/locobot_pan.stl"
             scale="0.001 0.001 0.001"/>
         </geometry>
@@ -105,5 +105,5 @@
         <geometry>
           <mesh
-            filename="package://interbotix_xslocobot_descriptions/meshes/locobot_meshes/locobot_tilt.stl"
+            filename="package://custom_locobot_description/meshes/locobot_meshes/locobot_tilt.stl"
             scale="0.001 0.001 0.001"/>
         </geometry>
@@ -116,5 +116,5 @@
         <geometry>
           <mesh
-            filename="package://interbotix_xslocobot_descriptions/meshes/locobot_meshes/locobot_tilt.stl"
+            filename="package://custom_locobot_description/meshes/locobot_meshes/locobot_tilt.stl"
             scale="0.001 0.001 0.001"/>
         </geometry>

File: urdf/kobuki_version/locobot_kobuki.urdf.xacro (robot description, xacro)
@@ -54,5 +54,5 @@
       <geometry>
         <mesh
-          filename="package://interbotix_xslocobot_descriptions/meshes/locobot_meshes/kobuki_version/kobuki.dae"/>
+          filename="package://custom_locobot_description/meshes/locobot_meshes/kobuki_version/kobuki.dae"/>
       </geometry>
     </visual>
@@ -122,5 +122,5 @@
       <geometry>
         <mesh
-          filename="package://interbotix_xslocobot_descriptions/meshes/locobot_meshes/kobuki_version/kobuki_wheel.dae"/>
+          filename="package://custom_locobot_description/meshes/locobot_meshes/kobuki_version/kobuki_wheel.dae"/>
       </geometry>
     </visual>
@@ -185,5 +185,5 @@
       <geometry>
         <mesh
-          filename="package://interbotix_xslocobot_descriptions/meshes/locobot_meshes/kobuki_version/kobuki_wheel.dae"/>
+          filename="package://custom_locobot_description/meshes/locobot_meshes/kobuki_version/kobuki_wheel.dae"/>
       </geometry>
     </visual>

File: urdf/lidar.urdf.xacro (robot description, xacro)
@@ -16,5 +16,5 @@
         <geometry>
           <mesh
-            filename="package://interbotix_xslocobot_descriptions/meshes/locobot_meshes/locobot_lidar_tower.stl"
+            filename="package://custom_locobot_description/meshes/locobot_meshes/locobot_lidar_tower.stl"
             scale="0.001 0.001 0.001"/>
         </geometry>
@@ -27,5 +27,5 @@
         <geometry>
           <mesh
-            filename="package://interbotix_xslocobot_descriptions/meshes/locobot_meshes/locobot_lidar_tower_simple.stl"
+            filename="package://custom_locobot_description/meshes/locobot_meshes/locobot_lidar_tower_simple.stl"
             scale="0.001 0.001 0.001"/>
         </geometry>
@@ -61,5 +61,5 @@
         <geometry>
           <mesh
-            filename="package://interbotix_xslocobot_descriptions/meshes/locobot_meshes/locobot_lidar.stl"
+            filename="package://custom_locobot_description/meshes/locobot_meshes/locobot_lidar.stl"
             scale="0.001 0.001 0.001"/>
         </geometry>

File: urdf/locobot.urdf.xacro (robot description, xacro)
@@ -22,10 +22,10 @@
     <texture filename="package://interbotix_common_sim/media/materials/textures/interbotix_black.png"/>
   </material>
-  <xacro:include filename="$(find interbotix_xslocobot_descriptions)/urdf/plate.urdf.xacro" />
-  <xacro:include filename="$(find interbotix_xslocobot_descriptions)/urdf/lidar.urdf.xacro" />
-  <xacro:include filename="$(find interbotix_xslocobot_descriptions)/urdf/battery.urdf.xacro" />
-  <xacro:include filename="$(find interbotix_xslocobot_descriptions)/urdf/arm_cradle.urdf.xacro" />
-  <xacro:include filename="$(find interbotix_xslocobot_descriptions)/urdf/camera_tower.urdf.xacro" />
-  <xacro:include filename="$(find interbotix_xslocobot_descriptions)/urdf/custom_pan_and_tilt.urdf.xacro" />
+  <xacro:include filename="$(find custom_locobot_description)/urdf/plate.urdf.xacro" />
+  <xacro:include filename="$(find custom_locobot_description)/urdf/lidar.urdf.xacro" />
+  <xacro:include filename="$(find custom_locobot_description)/urdf/battery.urdf.xacro" />
+  <xacro:include filename="$(find custom_locobot_description)/urdf/arm_cradle.urdf.xacro" />
+  <xacro:include filename="$(find custom_locobot_description)/urdf/camera_tower.urdf.xacro" />
+  <xacro:include filename="$(find custom_locobot_description)/urdf/custom_pan_and_tilt.urdf.xacro" />
   <link name="base_footprint"/>
   <xacro:if value="${arm_type == 'mobile_wx250s'}">
@@ -36,9 +36,9 @@
   </xacro:unless>
   <xacro:if value="${base_type == 'kobuki'}">
-    <xacro:include filename="$(find interbotix_xslocobot_descriptions)/urdf/kobuki_version/locobot_kobuki.urdf.xacro"/>
+    <xacro:include filename="$(find custom_locobot_description)/urdf/kobuki_version/locobot_kobuki.urdf.xacro"/>
     <xacro:property name="mesh_scale" value="0.001 0.001 0.001"/>
   </xacro:if> <!-- kobuki -->
   <xacro:if value="${base_type == 'create3'}">
-    <xacro:include filename="$(find interbotix_xslocobot_descriptions)/urdf/create3_version/locobot_create3.urdf.xacro"/>
+    <xacro:include filename="$(find custom_locobot_description)/urdf/create3_version/locobot_create3.urdf.xacro"/>
     <xacro:property name="mesh_scale" value="1 1 1"/>
   </xacro:if> <!-- create3 -->
@@ -86,5 +86,5 @@
   <!-- ********************************** Arm ********************************** -->
   <xacro:if value="${arm_type != 'mobile_base'}">
-    <xacro:include filename="$(find interbotix_xslocobot_descriptions)/urdf/arms/mobile_arm.urdf.xacro"/>
+    <xacro:include filename="$(find custom_locobot_description)/urdf/arms/mobile_arm.urdf.xacro"/>
     <xacro:mobile_arm/>
     <xacro:if value="${arm_type == 'mobile_wx200'}">

File: urdf/pan_and_tilt.urdf.xacro (robot description, xacro)
@@ -25,5 +25,5 @@
         <geometry>
           <mesh
-            filename="package://interbotix_xslocobot_descriptions/meshes/locobot_meshes/locobot_pan.stl"
+            filename="package://custom_locobot_description/meshes/locobot_meshes/locobot_pan.stl"
             scale="0.001 0.001 0.001"/>
         </geometry>
@@ -36,5 +36,5 @@
         <geometry>
           <mesh
-            filename="package://interbotix_xslocobot_descriptions/meshes/locobot_meshes/locobot_pan.stl"
+            filename="package://custom_locobot_description/meshes/locobot_meshes/locobot_pan.stl"
             scale="0.001 0.001 0.001"/>
         </geometry>
@@ -104,5 +104,5 @@
         <geometry>
           <mesh
-            filename="package://interbotix_xslocobot_descriptions/meshes/locobot_meshes/locobot_tilt.stl"
+            filename="package://custom_locobot_description/meshes/locobot_meshes/locobot_tilt.stl"
             scale="0.001 0.001 0.001"/>
         </geometry>
@@ -115,5 +115,5 @@
         <geometry>
           <mesh
-            filename="package://interbotix_xslocobot_descriptions/meshes/locobot_meshes/locobot_tilt.stl"
+            filename="package://custom_locobot_description/meshes/locobot_meshes/locobot_tilt.stl"
             scale="0.001 0.001 0.001"/>
         </geometry>
@@ -156,5 +156,5 @@
         <geometry>
           <mesh
-            filename="package://interbotix_xslocobot_descriptions/meshes/locobot_meshes/locobot_camera.stl"
+            filename="package://custom_locobot_description/meshes/locobot_meshes/locobot_camera.stl"
             scale="0.001 0.001 0.001"/>
         </geometry>
@@ -170,5 +170,5 @@
         <geometry>
           <mesh
-            filename="package://interbotix_xslocobot_descriptions/meshes/locobot_meshes/locobot_camera.stl"
+            filename="package://custom_locobot_description/meshes/locobot_meshes/locobot_camera.stl"
             scale="0.001 0.001 0.001"/>
         </geometry>

File: urdf/plate.urdf.xacro (robot description, xacro)
@@ -16,5 +16,5 @@
         <geometry>
           <mesh
-            filename="package://interbotix_xslocobot_descriptions/meshes/locobot_meshes/${base_type}_version/locobot_base_plate.stl"
+            filename="package://custom_locobot_description/meshes/locobot_meshes/${base_type}_version/locobot_base_plate.stl"
             scale="${mesh_scale}"/>
         </geometry>
@@ -27,5 +27,5 @@
         <geometry>
           <mesh
-            filename="package://interbotix_xslocobot_descriptions/meshes/locobot_meshes/${base_type}_version/locobot_base_plate.stl"
+            filename="package://custom_locobot_description/meshes/locobot_meshes/${base_type}_version/locobot_base_plate.stl"
             scale="${mesh_scale}"/>
         </geometry>

File: urdf/zed2.xacro (robot description, xacro)
@@ -15,10 +15,10 @@
       <visual>
         <geometry>
-          <mesh filename="package://interbotix_ros_descriptions/models/ZED2.dae"/>
+          <mesh filename="package://custom_locobot_description/models/ZED2.dae"/>
         </geometry>
       </visual>
       <collision>
         <geometry>
-          <mesh filename="package://interbotix_ros_descriptions/models/ZED2.dae"/>
+          <mesh filename="package://custom_locobot_description/models/ZED2.dae"/>
         </geometry>
       </collision>
