Commit message: Revert "add namespace robot_name to link"
This reverts commit c0e9bc735707d0d2719dccdfff4b584c29993600.

File: urdf/arm_cradle.urdf.xacro (robot description, xacro)
@@ -7,9 +7,9 @@
          <xacro:insert_block name="origin"/>
          <parent
-          link="${robot_name}/camera_tower_link"/>
+          link="camera_tower_link"/>
          <child
-          link="${robot_name}/arm_cradle_link"/>
+          link="arm_cradle_link"/>
       </joint>
-     <link name="${robot_name}/arm_cradle_link">
+     <link name="arm_cradle_link">
        <visual>
          <origin
@@ -49,5 +49,5 @@
       <disableFixedJointLumping>true</disableFixedJointLumping>
     </gazebo>
-    <gazebo reference="${robot_name}/arm_cradle_link">
+    <gazebo reference="arm_cradle_link">
       <material>Gazebo/DarkGrey</material>
     </gazebo>

File: urdf/battery.urdf.xacro (robot description, xacro)
@@ -5,9 +5,9 @@
       <xacro:insert_block name="origin"/>
       <parent
-        link="${robot_name}/plate_link"/>
+        link="plate_link"/>
       <child
-        link="${robot_name}/battery_link"/>
+        link="battery_link"/>
     </joint>
-    <link name="${robot_name}/battery_link">
+    <link name="battery_link">
       <visual>
         <origin
@@ -48,5 +48,5 @@
       </inertial>
     </link>
-    <gazebo reference="${robot_name}/battery_link">
+    <gazebo reference="battery_link">
       <material>Gazebo/Grey</material>
     </gazebo>

File: urdf/camera_tower.urdf.xacro (robot description, xacro)
@@ -5,9 +5,9 @@
       <xacro:insert_block name="origin"/>
       <parent
-        link="${robot_name}/base_link"/>
+        link="base_link"/>
       <child
-        link="${robot_name}/camera_tower_link"/>
+        link="camera_tower_link"/>
     </joint>
-    <link name="${robot_name}/camera_tower_link">
+    <link name="camera_tower_link">
       <visual>
         <origin
@@ -33,5 +33,5 @@
       <xacro:insert_block name="inertial"/>
     </link>
-    <gazebo reference="${robot_name}/camera_tower_link">
+    <gazebo reference="camera_tower_link">
       <material>Gazebo/DarkGrey</material>
     </gazebo>

File: urdf/custom_pan_and_tilt.urdf.xacro (robot description, xacro)
@@ -12,12 +12,12 @@
       <xacro:insert_block name="origin"/>
       <parent
-        link="${robot_name}/camera_tower_link"/>
+        link="camera_tower_link"/>
       <child
-        link="${robot_name}/pan_link"/>
+        link="pan_link"/>
       <dynamics
         friction="0.1"
         damping="0.1"/>
     </joint>
-    <link name="${robot_name}/pan_link">
+    <link name="pan_link">
       <visual>
         <origin
@@ -55,5 +55,5 @@
       </inertial>
     </link>
-    <gazebo reference="${robot_name}/pan_link">
+    <gazebo reference="pan_link">
       <material>Gazebo/DarkGrey</material>
       <self_collide>true</self_collide>
@@ -70,7 +70,7 @@
         xyz="0.025034 0 0.019"/>
       <parent
-        link="${robot_name}/pan_link"/>
+        link="pan_link"/>
       <child
-        link="${robot_name}/tilt_link"/>
+        link="tilt_link"/>
       <dynamics
         friction="0.1"
@@ -98,5 +98,5 @@
       </ros2_control>
     </xacro:if>
-    <link name="${robot_name}/tilt_link">
+    <link name="tilt_link">
       <visual>
         <origin
@@ -134,5 +134,5 @@
       </inertial>
     </link>
-    <gazebo reference="${robot_name}/tilt_link">
+    <gazebo reference="tilt_link">
       <material>Gazebo/DarkGrey</material>
       <self_collide>true</self_collide>
@@ -143,7 +143,7 @@
         xyz="0.05318 0.0175 0.000009"/>
       <parent
-        link="${robot_name}/tilt_link"/>
+        link="tilt_link"/>
       <child
-        link="${robot_name}/zed2_camera_center"/>
+        link="zed2_camera_center"/>
     </joint>
     <xacro:zed2/>

File: urdf/kobuki_version/locobot_kobuki.urdf.xacro (robot description, xacro)
@@ -43,9 +43,9 @@
       xyz="0 0 0.0102"/>
     <parent
-      link="${robot_name}/base_footprint"/>
-    <child
-      link="${robot_name}/base_link"/>
-  </joint>
-  <link name="${robot_name}/base_link">
+      link="base_footprint"/>
+    <child
+      link="base_link"/>
+  </joint>
+  <link name="base_link">
     <visual>
       <origin
@@ -99,7 +99,7 @@
       xyz="0.00 0.115 0.0250"/>
     <parent
-      link="${robot_name}/base_link"/>
-    <child
-      link="${robot_name}/wheel_left_link"/>
+      link="base_link"/>
+    <child
+      link="wheel_left_link"/>
   </joint>
   <xacro:if value="${hardware_type == 'gz_classic'}">
@@ -115,5 +115,5 @@
     </ros2_control>
   </xacro:if>
-  <link name="${robot_name}/wheel_left_link">
+  <link name="wheel_left_link">
     <visual>
       <origin
@@ -162,7 +162,7 @@
       xyz="0.00 -0.115 0.0250"/>
     <parent
-      link="${robot_name}/base_link"/>
-    <child
-      link="${robot_name}/wheel_right_link"/>
+      link="base_link"/>
+    <child
+      link="wheel_right_link"/>
   </joint>
   <xacro:if value="${hardware_type == 'gz_classic'}">
@@ -178,5 +178,5 @@
     </ros2_control>
   </xacro:if>
-  <link name="${robot_name}/wheel_right_link">
+  <link name="wheel_right_link">
     <visual>
       <origin
@@ -224,9 +224,9 @@
       xyz="0.115 0.0 0.007"/>
     <parent
-      link="${robot_name}/base_link"/>
-    <child
-      link="${robot_name}/caster_front_link"/>
-  </joint>
-  <link name="${robot_name}/caster_front_link">
+      link="base_link"/>
+    <child
+      link="caster_front_link"/>
+  </joint>
+  <link name="caster_front_link">
     <collision>
       <origin
@@ -265,9 +265,9 @@
       xyz="-0.135 0.0 0.009"/>
     <parent
-      link="${robot_name}/base_link"/>
-    <child
-      link="${robot_name}/caster_back_link"/>
-  </joint>
-  <link name="${robot_name}/caster_back_link">
+      link="base_link"/>
+    <child
+      link="caster_back_link"/>
+  </joint>
+  <link name="caster_back_link">
     <collision>
       <origin
@@ -306,9 +306,9 @@
       xyz="0.056 0.062 0.0202"/>
     <parent
-      link="${robot_name}/base_link"/>
-    <child
-      link="${robot_name}/gyro_link"/>
-  </joint>
-  <link name="${robot_name}/gyro_link">
+      link="base_link"/>
+    <child
+      link="gyro_link"/>
+  </joint>
+  <link name="gyro_link">
     <inertial>
       <origin
@@ -356,9 +356,9 @@
       xyz="0.08734 0.13601 0.0214"/>
     <parent
-      link="${robot_name}/base_link"/>
-    <child
-      link="${robot_name}/cliff_sensor_left_link"/>
-  </joint>
-  <link name="${robot_name}/cliff_sensor_left_link">
+      link="base_link"/>
+    <child
+      link="cliff_sensor_left_link"/>
+  </joint>
+  <link name="cliff_sensor_left_link">
     <inertial>
       <mass value="0.0001"/>
@@ -403,9 +403,9 @@
       xyz="0.085 -0.13601 0.0214"/>
     <parent
-      link="${robot_name}/base_link"/>
-    <child
-      link="${robot_name}/cliff_sensor_right_link"/>
-  </joint>
-  <link name="${robot_name}/cliff_sensor_right_link">
+      link="base_link"/>
+    <child
+      link="cliff_sensor_right_link"/>
+  </joint>
+  <link name="cliff_sensor_right_link">
     <inertial>
       <origin
@@ -450,9 +450,9 @@
       xyz="0.156 0.00 0.0214"/>
     <parent
-      link="${robot_name}/base_link"/>
-    <child
-      link="${robot_name}/cliff_sensor_front_link"/>
-  </joint>
-  <link name="${robot_name}/cliff_sensor_front_link">
+      link="base_link"/>
+    <child
+      link="cliff_sensor_front_link"/>
+  </joint>
+  <link name="cliff_sensor_front_link">
     <inertial>
       <mass value="0.0001"/>

File: urdf/lidar.urdf.xacro (robot description, xacro)
@@ -5,9 +5,9 @@
       <xacro:insert_block name="origin"/>
       <parent
-        link="${robot_name}/camera_tower_link"/>
+        link="camera_tower_link"/>
       <child
-        link="${robot_name}/lidar_tower_link"/>
+        link="lidar_tower_link"/>
     </joint>
-    <link name="${robot_name}/lidar_tower_link">
+    <link name="lidar_tower_link">
       <visual>
         <origin
@@ -50,9 +50,9 @@
         xyz="0 0 0.09425"/>
       <parent
-        link="${robot_name}/lidar_tower_link"/>
+        link="lidar_tower_link"/>
       <child
-        link="${robot_name}/laser_frame_link"/>
+        link="laser_frame_link"/>
     </joint>
-    <link name="${robot_name}/laser_frame_link">
+    <link name="laser_frame_link">
       <visual>
         <origin
@@ -90,5 +90,5 @@
       </inertial>
     </link>
-    <gazebo reference="${robot_name}/lidar_tower_link">
+    <gazebo reference="lidar_tower_link">
       <material>Gazebo/DarkGrey</material>
     </gazebo>
@@ -99,5 +99,5 @@
       <disableFixedJointLumping>true</disableFixedJointLumping>
     </gazebo>
-    <gazebo reference="${robot_name}/laser_frame_link">
+    <gazebo reference="laser_frame_link">
       <material>Gazebo/DarkGrey</material>
       <sensor type="ray" name="rplidar">
@@ -131,5 +131,5 @@
           </ros>
           <output_type>sensor_msgs/LaserScan</output_type>
-          <frame_name>${robot_name}/laser_frame_link</frame_name>
+          <frame_name>laser_frame_link</frame_name>
         </plugin>
       </sensor>

File: urdf/locobot.urdf.xacro (robot description, xacro)
@@ -3,5 +3,4 @@
   <xacro:arg name="arm_model"             default=""/>
   <xacro:arg name="robot_model"           default=""/>
-  <xacro:arg name="robot_name"            default=""/>
   <xacro:arg name="base_model"            default=""/>
   <xacro:arg name="show_lidar"            default="true"/>
@@ -14,5 +13,4 @@
   <xacro:property name="hardware_type"    value="$(arg hardware_type)"/>
   <xacro:property name="arm_type"         value="$(arg arm_model)"/>
-  <xacro:property name="robot_name"       value="$(arg robot_name)"/>
   <xacro:property name="base_type"        value="$(arg base_model)"/>
   <xacro:property name="urdf_loc"         value="$(arg external_urdf_loc)"/>
@@ -30,5 +28,5 @@
   <xacro:include filename="$(find custom_locobot_description)/urdf/camera_tower.urdf.xacro" />
   <xacro:include filename="$(find custom_locobot_description)/urdf/custom_pan_and_tilt.urdf.xacro" />
-  <link name="${robot_name}/base_footprint"/>
+  <link name="base_footprint"/>
   <xacro:if value="${arm_type == 'mobile_wx250s'}">
     <xacro:property name="camera_tower_size" value="large"/>

File: urdf/pan_and_tilt.urdf.xacro (robot description, xacro)
@@ -11,12 +11,12 @@
       <xacro:insert_block name="origin"/>
       <parent
-        link="${robot_name}/camera_tower_link"/>
+        link="camera_tower_link"/>
       <child
-        link="${robot_name}/pan_link"/>
+        link="pan_link"/>
       <dynamics
         friction="0.1"
         damping="0.1"/>
     </joint>
-    <link name="${robot_name}/pan_link">
+    <link name="pan_link">
       <visual>
         <origin
@@ -54,5 +54,5 @@
       </inertial>
     </link>
-    <gazebo reference="${robot_name}/pan_link">
+    <gazebo reference="pan_link">
       <material>Gazebo/DarkGrey</material>
       <self_collide>true</self_collide>
@@ -69,7 +69,7 @@
         xyz="0.025034 0 0.019"/>
       <parent
-        link="${robot_name}/pan_link"/>
+        link="pan_link"/>
       <child
-        link="${robot_name}/tilt_link"/>
+        link="tilt_link"/>
       <dynamics
         friction="0.1"
@@ -97,5 +97,5 @@
       </ros2_control>
     </xacro:if>
-    <link name="${robot_name}/tilt_link">
+    <link name="tilt_link">
       <visual>
         <origin
@@ -133,5 +133,5 @@
       </inertial>
     </link>
-    <gazebo reference="${robot_name}/tilt_link">
+    <gazebo reference="tilt_link">
       <material>Gazebo/DarkGrey</material>
       <self_collide>true</self_collide>
@@ -142,12 +142,12 @@
         xyz="0.05318 0.0175 0.000009"/>
       <parent
-        link="${robot_name}/tilt_link"/>
+        link="tilt_link"/>
       <child
-        link="${robot_name}/camera_link"/>
+        link="camera_link"/>
     </joint>
     <gazebo reference="camera">
       <disableFixedJointLumping>true</disableFixedJointLumping>
     </gazebo>
-    <link name="${robot_name}/camera_link">
+    <link name="camera_link">
       <visual>
         <origin
@@ -188,5 +188,5 @@
       </inertial>
     </link>
-    <gazebo reference="${robot_name}/camera_link">
+    <gazebo reference="camera_link">
       <material>Gazebo/Grey</material>
       <self_collide>true</self_collide>
@@ -196,11 +196,11 @@
     <joint name="camera_depth_joint" type="fixed">
       <origin rpy="${-pi/2} 0 ${-pi/2}" xyz="0 0 0"/>
-      <parent link="${robot_name}/camera_link"/>
-      <child link="${robot_name}/camera_depth_link"/>
-    </joint>
-    <link name="${robot_name}/camera_depth_link">
+      <parent link="camera_link"/>
+      <child link="camera_depth_link"/>
+    </joint>
+    <link name="camera_depth_link">
       <origin rpy="0 0 0" xyz="0 0 0"/>
     </link>
-    <gazebo reference="${robot_name}/camera_link">
+    <gazebo reference="camera_link">
       <sensor name="camera_frame_sensor" type="depth">
         <always_on>true</always_on>
@@ -227,5 +227,5 @@
           <depthImageCameraInfoTopicName>aligned_depth_to_color/camera_info</depthImageCameraInfoTopicName>
           <pointCloudTopicName>depth_registered/points</pointCloudTopicName>
-          <frameName>${robot_name}/camera_depth_link</frameName>
+          <frameName>camera_depth_link</frameName>
           <pointCloudCutoff>0.01</pointCloudCutoff>
           <pointCloudCutoffMax>10</pointCloudCutoffMax>

File: urdf/plate.urdf.xacro (robot description, xacro)
@@ -5,9 +5,9 @@
       <xacro:insert_block name="origin"/>
       <parent
-        link="${robot_name}/base_link"/>
+        link="base_link"/>
       <child
-        link="${robot_name}/plate_link"/>
+        link="plate_link"/>
     </joint>
-    <link name="${robot_name}/plate_link">
+    <link name="plate_link">
       <visual>
         <origin
@@ -33,5 +33,5 @@
       <xacro:insert_block name="inertial"/>
     </link>
-    <gazebo reference="${robot_name}/plate_link">
+    <gazebo reference="plate_link">
       <material>Gazebo/DarkGrey</material>
     </gazebo>

File: urdf/zed2.xacro (robot description, xacro)
@@ -2,7 +2,7 @@
 <robot xmlns:xacro="http://ros.org/wiki/xacro">
   <xacro:property name="baseline" value="0.12"/>
-  <xacro:macro name="zed2" params="origin">
+  <xacro:macro name="zed2">
     <!-- Camera Center -->
-    <link name="${robot_name}/zed2_camera_center">
+    <link name="zed2_camera_center">
       <inertial>
         <mass value="0.16140"/>
@@ -26,6 +26,6 @@
     <!-- Left Camera -->
     <joint name="zed2_left_camera_joint" type="fixed">
-      <parent link="${robot_name}/zed2_camera_center"/>
-      <child link="${robot_name}/zed2_left_camera_frame"/>
+      <parent link="zed2_camera_center"/>
+      <child link="zed2_left_camera_frame"/>
       <origin xyz="0 ${baseline/2} 0" rpy="0 0 0" />
     </joint>
@@ -33,46 +33,46 @@
     <joint name="zed2_left_camera_optical_joint" type="fixed">
       <origin xyz="0 0 0" rpy="-${pi/2} 0.0 -${pi/2}"/>
-      <parent link="${robot_name}/zed2_left_camera_frame"/>
-      <child link="${robot_name}/zed2_left_camera_optical_frame"/>
-    </joint>
-    <link name="${robot_name}/zed2_left_camera_optical_frame"/>
+      <parent link="zed2_left_camera_frame"/>
+      <child link="zed2_left_camera_optical_frame"/>
+    </joint>
+    <link name="zed2_left_camera_optical_frame"/>
     <!-- Right Camera -->
     <joint name="zed2_right_camera_joint" type="fixed">
-      <parent link="${robot_name}/zed2_camera_center"/>
-      <child link="${robot_name}/zed2_right_camera_frame"/>
+      <parent link="zed2_camera_center"/>
+      <child link="zed2_right_camera_frame"/>
       <origin xyz="0 -${baseline/2} 0" rpy="0 0 0" />
     </joint>
-    <link name="${robot_name}/zed2_right_camera_frame" />
+    <link name="zed2_right_camera_frame" />
     <joint name="zed2_right_camera_optical_joint" type="fixed">
       <origin xyz="0 0 0" rpy="-${pi/2} 0.0 -${pi/2}"/>
-      <parent link="${robot_name}/zed2_right_camera_frame"/>
-      <child link="${robot_name}/zed2_right_camera_optical_frame"/>
-    </joint>
-    <link name="${robot_name}/zed2_right_camera_optical_frame"/>
+      <parent link="zed2_right_camera_frame"/>
+      <child link="zed2_right_camera_optical_frame"/>
+    </joint>
+    <link name="zed2_right_camera_optical_frame"/>
     <!-- Sensors -->
     <joint name="zed2_mag_joint" type="fixed">
-      <parent link="${robot_name}/zed2_camera_center"/>
-      <child link="${robot_name}/zed2_mag_link"/>
+      <parent link="zed2_camera_center"/>
+      <child link="zed2_mag_link"/>
       <origin xyz="0 0 0" rpy="0 0 0" />
     </joint>
-    <link name="${robot_name}/zed2_mag_link" />
+    <link name="zed2_mag_link" />
     <joint name="zed2_baro_joint" type="fixed">
-      <parent link="${robot_name}/zed2_camera_center"/>
-      <child link="${robot_name}/zed2_baro_link"/>
+      <parent link="zed2_camera_center"/>
+      <child link="zed2_baro_link"/>
       <origin xyz="0 0 0" rpy="0 0 0" />
     </joint>
-    <link name="${robot_name}/zed2_baro_link" />
+    <link name="zed2_baro_link" />
     <joint name="zed2_temp_left_joint" type="fixed">
-      <parent link="${robot_name}/zed2_left_camera_frame"/>
-      <child link="${robot_name}/zed2_temp_left_link"/>
+      <parent link="zed2_left_camera_frame"/>
+      <child link="zed2_temp_left_link"/>
       <origin xyz="0 0 0" rpy="0 0 0" />
     </joint>
-    <link name="${robot_name}/zed2_temp_left_link" />
+    <link name="zed2_temp_left_link" />
     <joint name="zed2_temp_right_joint" type="fixed">
-        <parent link="${robot_name}/zed2_right_camera_frame"/>
-        <child link="${robot_name}/zed2_temp_right_link"/>
+        <parent link="zed2_right_camera_frame"/>
+        <child link="zed2_temp_right_link"/>
         <origin xyz="0 0 0" rpy="0 0 0" />
     </joint>
-    <link name="${robot_name}/zed2_temp_right_link" />
+    <link name="zed2_temp_right_link" />
   </xacro:macro>
   <xacro:macro name="zed2_gazebo">
